File: template-charlieplex_switches.kicad_sch (KiCad schematic)
At the start: 4 parts

Commit message: added footprints, misc fixes
Parts:
- DZD_: footprint (none) -> Package_TO_SOT_SMD:SOT-23-3
- D_: footprint (none) -> Diode_SMD:D_0201_0603Metric
Changed lines of the file:
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@@
 			)
 		)
-		(property "Footprint" ""
+		(property "Footprint" "Diode_SMD:D_0201_0603Metric"
 			(at 36.83 26.67 0)
 			(effects
@@
 			)
 		)
-		(property "Footprint" ""
+		(property "Footprint" "Package_TO_SOT_SMD:SOT-23-3"
 			(at 31.75 22.86 0)
 			(effects
